File: ruuvitag_revb3/ruuvitag_revb3.kicad_pcb (KiCad board)
At the start: 4 copper layers, 45 x 45 mm, 58 parts, among them P1 ARM_DEBUG, P10 TP, P11 TP, P12 TP, P13 TP, P14 TP, P15 TP, P16 TP, P17 TP, P18 TP, P19 TP, P2 TP, P20 TP, P21 TP, P22 TP, P23 TP, P3 TP, P4 NFC, P5 GND, P6 FIDUCIAL, P7 FIDUCIAL, P8 +BATT, P9 +BATT, Q1 Q_PMOS_GSD, SW1 SW_PUSH, SW2 SW_PUSH, U1 nRF52832, U2 BME280, U4 LIS2DH12, Y1 32K, Y2 32M

Commit message: DRC passed
Parts:
- added G***: G_LOGO, Ruuvi:G_LOGO, B.Cu at (86.5, 48.7)
- moved U4 0.59 mm to (63.1, 47.9)
- moved P10 0.50 mm to (72.5, 45.5)
- moved P11 0.25 mm to (69.8, 49.8)
Routing:
- net /SPI_MISO: track 20.9 -> 37.4 mm, vias 3 -> 5
- net /ACC_INT1: track 0.00 -> 14.3 mm, vias 0 -> 2
- net /ACC_INT2: track 0.00 -> 13.5 mm, vias 0 -> 2
- net GND: track 52.0 -> 54.5 mm
- net VDD: track 34.9 -> 35.8 mm
- net /SPI_SCK: track 27.2 -> 26.3 mm
- net /SWDIO: track 38.0 -> 37.2 mm
- net Net-(P10-Pad1): track 8.58 -> 7.89 mm
Other:
- net class Default: clearance 0.15 -> 0.149
- rule trace_clearance: 0.15 -> 0.149
